File: sensorBoard/Platine2.kicad_sch (KiCad schematic)
At the start: 14 parts, among them J17 Conn_01x04, J18 Conn_01x07, J19 Conn_01x03, J20 Conn_01x02, J21 Conn_01x04, J22 Conn_01x05, J23 Conn_01x02, U7 LD1117S33TR_SOT223

Commit message: aktualisierte Platine mit verschiedenen Stecker
Parts:
- removed J19: Conn_01x03, heder box:662103145021, symbol Connector_Generic:Conn_01x03
- removed J22: Conn_01x05, heder box:662105145021, symbol Connector_Generic:Conn_01x05
- removed J23: Conn_01x02, Connector_Phoenix_MC_HighVoltage:PhoenixContact_MCV_1,5_2-G-5.08_1x02_P5.08mm_Vertical, symbol Connector_Generic:Conn_01x02
- added J6, J7, J8: Conn_01x04, 6432101004xx:643210100404, symbol Connector_Generic:Conn_01x04
- J17: footprint Connector_Phoenix_MC_HighVoltage:PhoenixContact_MCV_1,5_4-G-5.08_1x04_P5.08mm_Vertical -> heder box:662104145021
- J21: footprint Connector_Phoenix_MC_HighVoltage:PhoenixContact_MCV_1,5_4-G-5.08_1x04_P5.08mm_Vertical -> 6432101004xx:643210100404
Connections:
- net +3.3V: now also J8.1 (Pin_1)
- net Commutation2-2/POLE+: now also J6.1 (Pin_1), J6.4 (Pin_4)
- net Commutation2-2/POLE-: now also J6.2 (Pin_2), J6.3 (Pin_3)
- net Commutation2-2/SERVO_OUT: now also J7.2 (Pin_2)
- net GND: now also J7.3 (Pin_3), J7.4 (Pin_4), J8.2 (Pin_2)
- net I2C_SCL: now also J8.3 (Pin_3)
- net I2C_SDA: now also J8.4 (Pin_4)
- net Protection2/12V_IN: now also J17.1 (Pin_1); no longer J17.4 (Pin_4)
- net Protection2/5V_IN: now also J17.4 (Pin_4); no longer J17.1 (Pin_1)
- net SERVO_PWM: now also J7.1 (Pin_1)
- net microcontroller2/UART_RX: now also J18.2 (Pin_2); no longer J18.1 (Pin_1)
- net microcontroller2/UART_TX: now also J18.1 (Pin_1); no longer J18.2 (Pin_2)
