File: sensorBoard/CanTransceiver.kicad_sch (KiCad schematic)
At the start: 4 parts, among them U3 MCP2551-I-SN

Commit message: added the footprints, connectors left
Parts:
- C13: footprint (none) -> Capacitor_SMD:C_0805_2012Metric
- R15, R16: footprint (none) -> Resistor_SMD:R_0805_2012Metric
Changed lines of the file:
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@@
 			)
 		)
-		(property "Footprint" ""
+		(property "Footprint" "Resistor_SMD:R_0805_2012Metric"
 			(at 116.84 96.52 0)
 			(effects
@@
 			)
 		)
-		(property "Footprint" ""
+		(property "Footprint" "Resistor_SMD:R_0805_2012Metric"
 			(at 154.94 85.09 0)
 			(effects
@@
 			)
 		)
-		(property "Footprint" ""
+		(property "Footprint" "Capacitor_SMD:C_0805_2012Metric"
 			(at 119.38 63.5 0)
 			(effects

Commit message: new two separate pcbs
Parts:
- renumbered C13 to C17, R15 to R33, R16 to R34, U3 to U12
Changed lines of the file:
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@@
 		(dnp no)
 		(fields_autoplaced yes)
-		(property "Reference" "R15"
+		(property "Reference" "R33"
 			(at 119.38 95.2499 0)
 			(effects
@@
 		)
 		(instances
-			(project ""
-				(path "/df1584e9-54f0-49dc-b423-5f64048efa01/f0fda8b3-f246-4adb-8696-ffc387bbcf07"
-					(reference "R15")
+			(project "sensorBoard"
+				(path "/df1584e9-54f0-49dc-b423-5f64048efa01/60fa4213-9bcb-42a7-994a-420953d9bcb7/92290787-937f-4ce6-9429-b8b9d4cb5373"
+					(reference "R17")
+					(unit 1)
+				)
+				(path "/df1584e9-54f0-49dc-b423-5f64048efa01/99847452-c15f-478e-a49b-00c0f2bcd04b/b58f972d-d58f-406a-9343-e3956f5ea2c8"
+					(reference "R33")
 					(unit 1)
 				)
@@
 		(dnp no)
 		(fields_autoplaced yes)
-		(property "Reference" "R16"
+		(property "Reference" "R34"
 			(at 157.48 83.8199 0)
 			(effects
@@
 		)
 		(instances
-			(project ""
-				(path "/df1584e9-54f0-49dc-b423-5f64048efa01/f0fda8b3-f246-4adb-8696-ffc387bbcf07"
-					(reference "R16")
+			(project "sensorBoard"
+				(path "/df1584e9-54f0-49dc-b423-5f64048efa01/60fa4213-9bcb-42a7-994a-420953d9bcb7/92290787-937f-4ce6-9429-b8b9d4cb5373"
+					(reference "R20")
+					(unit 1)
+				)
+				(path "/df1584e9-54f0-49dc-b423-5f64048efa01/99847452-c15f-478e-a49b-00c0f2bcd04b/b58f972d-d58f-406a-9343-e3956f5ea2c8"
+					(reference "R34")
 					(unit 1)
 				)
@@
 		(dnp no)
 		(fields_autoplaced yes)
-		(property "Reference" "#PWR040"
+		(property "Reference" "#PWR090"
 			(at 135.89 59.69 0)
 			(effects
@@
 		)
 		(instances
-			(project ""
-				(path "/df1584e9-54f0-49dc-b423-5f64048efa01/f0fda8b3-f246-4adb-8696-ffc387bbcf07"
-					(reference "#PWR040")
+			(project "sensorBoard"
+				(path "/df1584e9-54f0-49dc-b423-5f64048efa01/60fa4213-9bcb-42a7-994a-420953d9bcb7/92290787-937f-4ce6-9429-b8b9d4cb5373"
+					(reference "#PWR0190")
+					(unit 1)
+				)
+				(path "/df1584e9-54f0-49dc-b423-5f64048efa01/99847452-c15f-478e-a49b-00c0f2bcd04b/b58f972d-d58f-406a-9343-e3956f5ea2c8"
+					(reference "#PWR090")
 					(unit 1)
 				)
@@
 		(dnp no)
 		(fields_autoplaced yes)
-		(property "Reference" "C13"
+		(property "Reference" "C17"
 			(at 121.92 62.2362 0)
 			(effects
@@
 		)
 		(instances
-			(project ""
-				(path "/df1584e9-54f0-49dc-b423-5f64048efa01/f0fda8b3-f246-4adb-8696-ffc387bbcf07"
-					(reference "C13")
+			(project "sensorBoard"
+				(path "/df1584e9-54f0-49dc-b423-5f64048efa01/60fa4213-9bcb-42a7-994a-420953d9bcb7/92290787-937f-4ce6-9429-b8b9d4cb5373"
+					(reference "C39")
+					(unit 1)
+				)
+				(path "/df1584e9-54f0-49dc-b423-5f64048efa01/99847452-c15f-478e-a49b-00c0f2bcd04b/b58f972d-d58f-406a-9343-e3956f5ea2c8"
+					(reference "C17")
 					(unit 1)
 				)
@@
 		(dnp no)
 		(fields_autoplaced yes)
-		(property "Reference" "#PWR039"
+		(property "Reference" "#PWR054"
 			(at 116.84 109.22 0)
 			(effects
@@
 		)
 		(instances
-			(project ""
-				(path "/df1584e9-54f0-49dc-b423-5f64048efa01/f0fda8b3-f246-4adb-8696-ffc387bbcf07"
-					(reference "#PWR039")
+			(project "sensorBoard"
+				(path "/df1584e9-54f0-49dc-b423-5f64048efa01/60fa4213-9bcb-42a7-994a-420953d9bcb7/92290787-937f-4ce6-9429-b8b9d4cb5373"
+					(reference "#PWR0188")
+					(unit 1)
+				)
+				(path "/df1584e9-54f0-49dc-b423-5f64048efa01/99847452-c15f-478e-a49b-00c0f2bcd04b/b58f972d-d58f-406a-9343-e3956f5ea2c8"
+					(reference "#PWR054")
 					(unit 1)
 				)
@@
 		(dnp no)
 		(fields_autoplaced yes)
-		(property "Reference" "#PWR042"
+		(property "Reference" "#PWR091"
 			(at 135.89 109.22 0)
 			(effects
@@
 		)
 		(instances
-			(project ""
-				(path "/df1584e9-54f0-49dc-b423-5f64048efa01/f0fda8b3-f246-4adb-8696-ffc387bbcf07"
-					(reference "#PWR042")
+			(project "sensorBoard"
+				(path "/df1584e9-54f0-49dc-b423-5f64048efa01/60fa4213-9bcb-42a7-994a-420953d9bcb7/92290787-937f-4ce6-9429-b8b9d4cb5373"
+					(reference "#PWR0191")
+					(unit 1)
+				)
+				(path "/df1584e9-54f0-49dc-b423-5f64048efa01/99847452-c15f-478e-a49b-00c0f2bcd04b/b58f972d-d58f-406a-9343-e3956f5ea2c8"
+					(reference "#PWR091")
 					(unit 1)
 				)
@@
 		(on_board yes)
 		(dnp no)
-		(property "Reference" "U3"
+		(property "Reference" "U12"
 			(at 138.43 72.39 0)
 			(effects
@@
 		)
 		(instances
-			(project ""
-				(path "/df1584e9-54f0-49dc-b423-5f64048efa01/f0fda8b3-f246-4adb-8696-ffc387bbcf07"
-					(reference "U3")
+			(project "sensorBoard"
+				(path "/df1584e9-54f0-49dc-b423-5f64048efa01/60fa4213-9bcb-42a7-994a-420953d9bcb7/92290787-937f-4ce6-9429-b8b9d4cb5373"
+					(reference "U9")
+					(unit 1)
+				)
+				(path "/df1584e9-54f0-49dc-b423-5f64048efa01/99847452-c15f-478e-a49b-00c0f2bcd04b/b58f972d-d58f-406a-9343-e3956f5ea2c8"
+					(reference "U12")
 					(unit 1)
 				)
@@
 		(dnp no)
 		(fields_autoplaced yes)
-		(property "Reference" "#PWR041"
+		(property "Reference" "#PWR072"
 			(at 119.38 74.93 0)
 			(effects
@@
 		)
 		(instances
-			(project ""
-				(path "/df1584e9-54f0-49dc-b423-5f64048efa01/f0fda8b3-f246-4adb-8696-ffc387bbcf07"
-					(reference "#PWR041")
-					(unit 1)
-				)
+			(project "sensorBoard"
+				(path "/df1584e9-54f0-49dc-b423-5f64048efa01/60fa4213-9bcb-42a7-994a-420953d9bcb7/92290787-937f-4ce6-9429-b8b9d4cb5373"
+					(reference "#PWR0189")
+					(unit 1)
+				)
+				(path "/df1584e9-54f0-49dc-b423-5f64048efa01/99847452-c15f-478e-a49b-00c0f2bcd04b/b58f972d-d58f-406a-9343-e3956f5ea2c8"
+					(reference "#PWR072")
+					(unit 1)
+				)

Commit message: Das erstes PCB ist fast fertig. Die Vias waren auf die Platine platziert und Poligon war gefüllt.
Parts:
- renumbered C17 to C39, R33 to R17, R34 to R20, U12 to U9
Changed lines of the file:
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@@
 		(dnp no)
 		(fields_autoplaced yes)
-		(property "Reference" "R33"
+		(property "Reference" "R17"
 			(at 119.38 95.2499 0)
 			(effects
@@
 		(dnp no)
 		(fields_autoplaced yes)
-		(property "Reference" "R34"
+		(property "Reference" "R20"
 			(at 157.48 83.8199 0)
 			(effects
@@
 		(dnp no)
 		(fields_autoplaced yes)
-		(property "Reference" "#PWR090"
+		(property "Reference" "#PWR0190"
 			(at 135.89 59.69 0)
 			(effects
@@
 		(dnp no)
 		(fields_autoplaced yes)
-		(property "Reference" "C17"
+		(property "Reference" "C39"
 			(at 121.92 62.2362 0)
 			(effects
@@
 		(dnp no)
 		(fields_autoplaced yes)
-		(property "Reference" "#PWR054"
+		(property "Reference" "#PWR0188"
 			(at 116.84 109.22 0)
 			(effects
@@
 		(dnp no)
 		(fields_autoplaced yes)
-		(property "Reference" "#PWR091"
+		(property "Reference" "#PWR0191"
 			(at 135.89 109.22 0)
 			(effects
@@
 		(on_board yes)
 		(dnp no)
-		(property "Reference" "U12"
+		(property "Reference" "U9"
 			(at 138.43 72.39 0)
 			(effects
@@
 		(dnp no)
 		(fields_autoplaced yes)
-		(property "Reference" "#PWR072"
+		(property "Reference" "#PWR0189"
 			(at 119.38 74.93 0)
 			(effects

Commit message: added old software + new PCB
Parts:
- removed U9: MCP2551-I-SN, Package_SO:SOIC-8_3.9x4.9mm_P1.27mm, symbol Interface_CAN_LIN:MCP2551-I-SN
- added SW1: SW_DIP_x01, Pavel_library:416131160801, symbol Switch:SW_DIP_x01
- added U2: MAX3051, Package_SO:SOIC-8_3.9x4.9mm_P1.27mm, symbol Interface_UART:MAX3051
- R33: renamed from R17; value R_Small -> 0
- renumbered C39 to C17, R20 to R34
Connections:
- net CAN_H: now also R34.2, U2.7 (CANH); no longer R34.1
- net CAN_L: now also SW1.2, U2.6 (CANL); no longer R34.2
- net CAN_RX: now also U2.4 (RXD)
- net CAN_TX: now also U2.1 (TXD)
- net GND: now also U2.2 (GND)
- net at R33.1: now also U2.8 (RS)
- net +5V renamed +3.3V
- net +3.3V: now also U2.3 (VDD)
- new net: R34.1, SW1.1
Other:
- moved on the sheet: R34
