File: sensorBoard/Motor_driver_1-1.kicad_sch (KiCad schematic)
At the start: 9 parts, among them K3 G2RL-1-H, K4 G2RL-1-H, Q8 2N7002, Q9 2N7002, U14 4011, U24 4011

Commit message: new two separate pcbs
Parts:
- renumbered D4 to D22, D5 to D23, K3 to K5, K4 to K6, Q8 to Q21, Q9 to Q22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
